Commit message: Added everything until object racking

File: description/camera.xacro (robot description, xacro)
@@ -4,5 +4,5 @@
         <parent link="chassis"/>
         <child link="camera_link"/>
-        <origin xyz="0.305 0.0 0.08" rpy="0.0 0.0 0.0"/>
+        <origin xyz="0.305 0.0 0.08" rpy="0.0 0.18 0.0"/>
     </joint>
     <link name="camera_link">

File: description/robot_core.xacro (robot description, xacro)
@@ -18,4 +18,10 @@
     </material>
     <link name = "base_link">
+    </link>
+    <joint name="footprint_joint" type="fixed">
+        <parent link="base_link"/>
+        <child link="base_footprint"/>
+    </joint>
+    <link name="base_footprint">
     </link>
     <joint name="chassis_joint" type="fixed">
